File: kicad/dropphoto.kicad_pcb (KiCad board)
At the start: 2 copper layers, 34 parts, among them J1 Conn_01x02, J2 Conn_01x02, J3 Conn_01x02, J4 Conn_01x02, J5 Conn_01x03, J6 Conn_01x03, J7 Conn_01x02, Q1 IRFZ44N, Q2 IRFZ44N, U1 Arduino_Nano_v3.x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

Commit message: Finish routing.
Parts:
- removed J5, J6: Conn_01x03, Connector_JST:JST_XH_B03B-XH-A_1x03_P2.50mm_Vertical
- added REF**: MountingHole_10mm, MountingHole:MountingHole_10mm, F.Cu at (31.1, 80.0)
- added REF**: MountingHole_3.2mm_M3, MountingHole:MountingHole_3.2mm_M3, F.Cu at (22.9, 101.6)
- added REF**: MountingHole_3.2mm_M3, MountingHole:MountingHole_3.2mm_M3, F.Cu at (22.9, 61.0)
- added REF**: MountingHole_3.2mm_M3, MountingHole:MountingHole_3.2mm_M3, F.Cu at (99.7, 61.0)
- added REF**: MountingHole_3.2mm_M3, MountingHole:MountingHole_3.2mm_M3, F.Cu at (157.5, 102.2)
- JP1, R7: moved to B.Cu
- moved U2 226.6 mm to (110.5, 73.0)
- moved C5 224.7 mm to (108.6, 66.7)
- moved D3 224.7 mm to (139.7, 73.0)
- moved R7 224.7 mm to (151.8, 79.0), turned to 90 degrees
- moved C7 224.7 mm to (132.7, 66.7)
- moved JP1 224.7 mm to (148.6, 78.7), turned to 90 degrees
- moved Q1 224.7 mm to (156.2, 71.1)
- moved R4 224.7 mm to (128.9, 78.7)
- moved C6 224.7 mm to (118.7, 66.7)
- moved C8 224.7 mm to (146.7, 66.7)
- moved J1 224.7 mm to (158.1, 60.3)
- moved J2 224.7 mm to (158.1, 83.8)
- moved C4 191.0 mm to (104.8, 75.6), turned to 270 degrees
- moved C3 185.7 mm to (99.7, 75.6), turned to 270 degrees
- moved R5 76.3 mm to (110.5, 102.9)
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Connections:
- D2 pad 1: Net-(D2-Pad1) -> OPTO
- R2 pad 2: Net-(D2-Pad1) -> OPTO
- U1 pad 8: Net-(J5-Pad2) -> OPTO
- U3 pad 1: Net-(J3-Pad2) -> Net-(J3-Pad1)
- U3 pad 2: Net-(J3-Pad1) -> Net-(J3-Pad2)
Routing:
- net GND: track 0.00 -> 397.1 mm, vias 0 -> 4
- net +5V: track 0.00 -> 136.2 mm, vias 0 -> 2
- net +12V: track 0.00 -> 125.8 mm, vias 0 -> 2
- net TRIG: track 0.00 -> 103.5 mm, vias 0 -> 2
- net Net-(C5-Pad1): track 0.00 -> 82.0 mm, vias 0 -> 2
- net PUMP: track 0.00 -> 78.4 mm, vias 0 -> 2
- net SHUTTER: track 0.00 -> 71.1 mm
- net OPTO: track 0.00 -> 50.4 mm
- net Net-(Q1-Pad1): track 0.00 -> 45.3 mm
- net +BATT: track 0.00 -> 26.6 mm
- net Net-(J2-Pad1): track 0.00 -> 20.7 mm
- net Net-(D3-Pad2): track 0.00 -> 18.0 mm
- net Net-(D4-Pad2): track 0.00 -> 14.0 mm
- net Net-(J3-Pad2): track 0.00 -> 11.7 mm
- net Net-(Q2-Pad1): track 0.00 -> 10.6 mm
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Other:
- board outline added: 142.2 x 49.5 mm
- net class Default: clearance 0.2 -> 0.5; trace_width 0.25 -> 1; via_dia 0.8 -> 3; via_drill 0.4 -> 1
- rule trace_clearance: 0.2 -> 0.5
