File: kicad/dropphoto.sch (KiCad schematic (older format))
At the start: 18 parts

Commit message: Complete diagram.
Parts:
- removed Q?: Q_NMOS_DGS, symbol Device:Q_NMOS_DGS
- added C1: 470n, symbol Device:C
- added C2: 100n, symbol Device:C
- added D4: 1N4001, symbol Device:D_ALT
- added J3, J4: Conn_01x02, symbol Connector_Generic:Conn_01x02
- added JP1: CM, symbol Jumper:SolderJumper_2_Bridged
- added Q1, Q2: IRFZ44N, symbol Device:Q_NMOS_GDS
- added R2: 15k, symbol Device:R
- added R5: 1k, symbol Device:R
- added R6: 47k, symbol Device:R
- added U3: 4066, symbol 4xxx:4066
- added U4: LM7812_TO220, Package_TO_SOT_THT:TO-220-3_Vertical, symbol Regulator_Linear:LM7812_TO220
- D1: renamed from D?; value LED_ALT -> 455.IRT
- D2: renamed from D?; value D_Photo_ALT -> 455.IRR
- D3: renamed from D?; value D_ALT -> 1N4001
- R1: renamed from R?; value R -> 220
- R7: renamed from R?; value 0R02 -> 0R01
- gave numbers to parts that had none: 12
Connections:
- net +5V: now also U1.27 (+5V), R2.1, U3.12, U3.14 (VDD)
- net +BATT: now also C1.1, U4.1 (VI)
- net GND: now also D2.2 (A), U1.29 (GND), U1.4 (GND), C1.2, C2.2, JP1.2 (B), Q2.3 (S), R6.1, U3.5, U3.6, U3.7 (VSS), U4.2 (GND)
- net TRIG: now also U1.8 (D5)
- net at R4.1, U2.6 (OUTPUT_2), U2.7 (OUTPUT): now also Q1.1 (G)
- net +12V: now reaches U1.30 (VIN)
- net +12V: now also C2.1, D4.1 (K), J4.1 (Pin_1), U4.3 (VO)
- net PUMP: now reaches U1.6 (D3)
- net PUMP: now also R5.2, R6.2
- net SHUTTER: now reaches U1.7 (D4)
- net SHUTTER: now also U3.13
- net at U1.9 (D6): now also D2.1 (K), R2.2
- net at D3.2 (A), J1.2 (Pin_2): now also Q1.2 (D)
- net at J2.1 (Pin_1), R7.1: now also JP1.1 (A), Q1.3 (S)
- new net: D4.2 (A), J4.2 (Pin_2), Q2.2 (D)
- new net: J3.2 (Pin_2), U3.1
- new net: J3.1 (Pin_1), U3.2
- new net: Q2.1 (G), R5.1
- no-connect marks 0 -> 28
Other:
- note added: "Current measurement"
- note added: "LEDs"
- note added: "Pump"
- note added: "Shutter"

Commit message: Fix errors.
Parts:
- added C9: 1u, symbol Device:C
- added J5, J6: Conn_01x03, symbol Connector_Generic:Conn_01x03
- added J7: Conn_01x02, symbol Connector_Generic:Conn_01x02
Connections:
- net +12V: now also C3.1, C4.1, U2.1 (VDD_2), U2.8 (VDD)
- net +5V: now also C9.1, J5.1 (Pin_1), J6.1 (Pin_1)
- net +BATT: now also J7.1 (Pin_1)
- net GND: now also C9.2, J5.3 (Pin_3), J6.3 (Pin_3), J7.2 (Pin_2)
- net TRIG: now also U1.9 (D6); no longer U1.8 (D5)
- net at D2.1 (K), R2.2: now also J6.2 (Pin_2); no longer U1.9 (D6)
- new net: J5.2 (Pin_2), U1.8 (D5)
Other:
- note added: "OPTO"
- moved on the sheet: D1, D2, R1, R2

Commit message: Start defining footprints.
Parts:
- D1, D2: footprint (none) -> LED_THT:LED_D5.0mm_Horizontal_O1.27mm_Z3.0mm_IRBlack
- D3, D4: footprint (none) -> Diode_THT:D_A-405_P12.70mm_Horizontal
- J1, J2, J3, J4, J7: footprint (none) -> Connector_JST:JST_XH_B02B-XH-A_1x02_P2.50mm_Vertical
- J5, J6: footprint (none) -> Connector_JST:JST_XH_B03B-XH-A_1x03_P2.50mm_Vertical
- JP1: footprint (none) -> Jumper:SolderJumper-2_P1.3mm_Bridged_RoundedPad1.0x1.5mm
- Q1, Q2: footprint (none) -> Package_TO_SOT_THT:TO-220-3_Vertical
- R1, R2, R3, R4, R5, R6: footprint (none) -> Resistor_THT:R_Axial_DIN0414_L11.9mm_D4.5mm_P15.24mm_Horizontal
- R7: footprint (none) -> Resistor_SMD:R_2512_6332Metric
- U2: footprint DIP254P762X533-8 -> Package_DIP:DIP-8_W7.62mm_LongPads
- U3: footprint (none) -> Package_DIP:DIP-14_W7.62mm_LongPads
Changed lines of the file:
@@
 F 0 "U2" H 5700 3570 50  0000 C CNN
 F 1 "TC4420CPA" H 5700 3479 50  0000 C CNN
-F 2 "DIP254P762X533-8" H 5700 3100 50  0001 L BNN
+F 2 "Package_DIP:DIP-8_W7.62mm_LongPads" H 5700 3100 50  0001 L BNN
 F 3 "" H 5700 3100 50  0001 L BNN
 F 4 "None" H 5700 3100 50  0001 L BNN "Field4"
@@
 F 0 "J1" H 9230 2542 50  0000 L CNN
 F 1 "Conn_01x02" H 9230 2451 50  0000 L CNN
-F 2 "" H 9150 2550 50  0001 C CNN
+F 2 "Connector_JST:JST_XH_B02B-XH-A_1x02_P2.50mm_Vertical" H 9150 2550 50  0001 C CNN
 F 3 "~" H 9150 2550 50  0001 C CNN
 	1    9150 2550
@@
 F 0 "D1" V 5100 5450 50  0000 R CNN
 F 1 "455.IRT" V 4950 5550 50  0000 R CNN
-F 2 "" H 5100 5200 50  0001 C CNN
+F 2 "LED_THT:LED_D5.0mm_Horizontal_O1.27mm_Z3.0mm_IRBlack" H 5100 5200 50  0001 C CNN
 F 3 "~" H 5100 5200 50  0001 C CNN
 	1    5100 5200
@@
 F 0 "R1" H 5170 4796 50  0000 L CNN
 F 1 "220" H 5170 4705 50  0000 L CNN
-F 2 "" V 5030 4750 50  0001 C CNN
+F 2 "Resistor_THT:R_Axial_DIN0414_L11.9mm_D4.5mm_P15.24mm_Horizontal" V 5030 4750 50  0001 C CNN
 F 3 "~" H 5100 4750 50  0001 C CNN
 	1    5100 4750
@@
 F 0 "R4" H 7670 3746 50  0000 L CNN
 F 1 "47k" H 7670 3655 50  0000 L CNN
-F 2 "" V 7530 3700 50  0001 C CNN
+F 2 "Resistor_THT:R_Axial_DIN0414_L11.9mm_D4.5mm_P15.24mm_Horizontal" V 7530 3700 50  0001 C CNN
 F 3 "~" H 7600 3700 50  0001 C CNN
 	1    7600 3700
@@
 F 0 "R7" H 8520 3746 50  0000 L CNN
 F 1 "0R01" H 8520 3655 50  0000 L CNN
-F 2 "" V 8380 3700 50  0001 C CNN
+F 2 "Resistor_SMD:R_2512_6332Metric" V 8380 3700 50  0001 C CNN
 F 3 "~" H 8450 3700 50  0001 C CNN
 	1    8450 3700
@@
 F 0 "D3" V 8404 2729 50  0000 L CNN
 F 1 "1N4001" V 8495 2729 50  0000 L CNN
-F 2 "" H 8450 2650 50  0001 C CNN
+F 2 "Diode_THT:D_A-405_P12.70mm_Horizontal" H 8450 2650 50  0001 C CNN
 F 3 "~" H 8450 2650 50  0001 C CNN
 	1    8450 2650
@@
 F 0 "R3" V 5943 2350 50  0000 C CNN
 F 1 "100" V 6034 2350 50  0000 C CNN
-F 2 "" V 6080 2350 50  0001 C CNN
+F 2 "Resistor_THT:R_Axial_DIN0414_L11.9mm_D4.5mm_P15.24mm_Horizontal" V 6080 2350 50  0001 C CNN
 F 3 "~" H 6150 2350 50  0001 C CNN
 	1    6150 2350
@@
 F 0 "J2" H 9230 3642 50  0000 L CNN
 F 1 "Conn_01x02" H 9230 3551 50  0000 L CNN
-F 2 "" H 9150 3650 50  0001 C CNN
+F 2 "Connector_JST:JST_XH_B02B-XH-A_1x02_P2.50mm_Vertical" H 9150 3650 50  0001 C CNN
 F 3 "~" H 9150 3650 50  0001 C CNN
 	1    9150 3650
@@
 F 0 "J3" H 9230 4892 50  0000 L CNN
 F 1 "Conn_01x02" H 9230 4801 50  0000 L CNN
-F 2 "" H 9150 4900 50  0001 C CNN
+F 2 "Connector_JST:JST_XH_B02B-XH-A_1x02_P2.50mm_Vertical" H 9150 4900 50  0001 C CNN
 F 3 "~" H 9150 4900 50  0001 C CNN
 	1    9150 4900
@@
 F 0 "JP1" V 8104 3768 50  0000 L CNN
 F 1 "CM" V 8195 3768 50  0000 L CNN
-F 2 "" H 8150 3700 50  0001 C CNN
+F 2 "Jumper:SolderJumper-2_P1.3mm_Bridged_RoundedPad1.0x1.5mm" H 8150 3700 50  0001 C CNN
 F 3 "~" H 8150 3700 50  0001 C CNN
 	1    8150 3700
@@
 F 0 "J4" H 9230 5642 50  0000 L CNN
 F 1 "Conn_01x02" H 9230 5551 50  0000 L CNN
-F 2 "" H 9150 5650 50  0001 C CNN
+F 2 "Connector_JST:JST_XH_B02B-XH-A_1x02_P2.50mm_Vertical" H 9150 5650 50  0001 C CNN
 F 3 "~" H 9150 5650 50  0001 C CNN
 	1    9150 5650
@@
 F 0 "D4" V 8454 5729 50  0000 L CNN
 F 1 "1N4001" V 8545 5729 50  0000 L CNN
-F 2 "" H 8500 5650 50  0001 C CNN
+F 2 "Diode_THT:D_A-405_P12.70mm_Horizontal" H 8500 5650 50  0001 C CNN
 F 3 "~" H 8500 5650 50  0001 C CNN
 	1    8500 5650
@@
 F 0 "R5" V 8043 6100 50  0000 C CNN
 F 1 "1k" V 8134 6100 50  0000 C CNN
-F 2 "" V 8180 6100 50  0001 C CNN
+F 2 "Resistor_THT:R_Axial_DIN0414_L11.9mm_D4.5mm_P15.24mm_Horizontal" V 8180 6100 50  0001 C CNN
 F 3 "~" H 8250 6100 50  0001 C CNN
 	1    8250 6100
@@
 F 0 "R6" V 8150 6150 50  0000 C CNN
 F 1 "47k" V 8134 6350 50  0000 C CNN
-F 2 "" V 8180 6350 50  0001 C CNN
+F 2 "Resistor_THT:R_Axial_DIN0414_L11.9mm_D4.5mm_P15.24mm_Horizontal" V 8180 6350 50  0001 C CNN
 F 3 "~" H 8250 6350 50  0001 C CNN
 	1    8250 6350
@@
 F 0 "U3" H 7950 4727 50  0000 C CNN
 F 1 "4066" H 7950 4636 50  0000 C CNN
-F 2 "" H 7950 4900 50  0001 C CNN
+F 2 "Package_DIP:DIP-14_W7.62mm_LongPads" H 7950 4900 50  0001 C CNN
 F 3 "http://www.ti.com/lit/ds/symlink/cd4066b.pdf" H 7950 4900 50  0001 C CNN
 	1    7950 4900
@@
 F 0 "R2" H 5720 4796 50  0000 L CNN
 F 1 "15k" H 5720 4705 50  0000 L CNN
-F 2 "" V 5580 4750 50  0001 C CNN
+F 2 "Resistor_THT:R_Axial_DIN0414_L11.9mm_D4.5mm_P15.24mm_Horizontal" V 5580 4750 50  0001 C CNN
 F 3 "~" H 5650 4750 50  0001 C CNN
 	1    5650 4750
@@
 F 0 "Q1" H 8556 3246 50  0000 L CNN
 F 1 "IRFZ44N" H 8556 3155 50  0000 L CNN
-F 2 "" H 8550 3300 50  0001 C CNN
+F 2 "Package_TO_SOT_THT:TO-220-3_Vertical" H 8550 3300 50  0001 C CNN
 F 3 "~" H 8350 3200 50  0001 C CNN
 	1    8350 3200
@@
 F 0 "Q2" H 8956 6146 50  0000 L CNN
 F 1 "IRFZ44N" H 8956 6055 50  0000 L CNN
-F 2 "" H 8950 6200 50  0001 C CNN
+F 2 "Package_TO_SOT_THT:TO-220-3_Vertical" H 8950 6200 50  0001 C CNN
 F 3 "~" H 8750 6100 50  0001 C CNN
 	1    8750 6100
@@
 F 0 "U3" H 2700 6627 50  0000 C CNN
 F 1 "4066" H 2700 6536 50  0000 C CNN
-F 2 "" H 2700 6800 50  0001 C CNN
+F 2 "Package_DIP:DIP-14_W7.62mm_LongPads" H 2700 6800 50  0001 C CNN
 F 3 "http://www.ti.com/lit/ds/symlink/cd4066b.pdf" H 2700 6800 50  0001 C CNN
 	3    2700 6800
@@
 F 0 "U3" H 1700 6627 50  0000 C CNN
 F 1 "4066" H 1700 6536 50  0000 C CNN
-F 2 "" H 1700 6800 50  0001 C CNN
+F 2 "Package_DIP:DIP-14_W7.62mm_LongPads" H 1700 6800 50  0001 C CNN
 F 3 "http://www.ti.com/lit/ds/symlink/cd4066b.pdf" H 1700 6800 50  0001 C CNN
 	2    1700 6800
@@
 F 0 "U3" H 3650 6627 50  0000 C CNN
 F 1 "4066" H 3650 6536 50  0000 C CNN
-F 2 "" H 3650 6800 50  0001 C CNN
+F 2 "Package_DIP:DIP-14_W7.62mm_LongPads" H 3650 6800 50  0001 C CNN
 F 3 "http://www.ti.com/lit/ds/symlink/cd4066b.pdf" H 3650 6800 50  0001 C CNN
 	4    3650 6800
@@
 F 0 "U3" H 4880 6846 50  0000 L CNN
 F 1 "4066" H 4880 6755 50  0000 L CNN
-F 2 "" H 4650 6800 50  0001 C CNN
+F 2 "Package_DIP:DIP-14_W7.62mm_LongPads" H 4650 6800 50  0001 C CNN
 F 3 "http://www.ti.com/lit/ds/symlink/cd4066b.pdf" H 4650 6800 50  0001 C CNN
 	5    4650 6800
@@
 F 0 "D2" V 5550 5050 50  0000 L CNN
 F 1 "455.IRR" V 5700 4950 50  0000 L CNN
-F 2 "" H 5600 5350 50  0001 C CNN
+F 2 "LED_THT:LED_D5.0mm_Horizontal_O1.27mm_Z3.0mm_IRBlack" H 5600 5350 50  0001 C CNN
 F 3 "~" H 5600 5350 50  0001 C CNN
 	1    5650 5350
@@
 F 0 "J6" H 6630 5092 50  0000 L CNN
 F 1 "Conn_01x03" H 6630 5001 50  0000 L CNN
-F 2 "" H 6550 5050 50  0001 C CNN
+F 2 "Connector_JST:JST_XH_B03B-XH-A_1x03_P2.50mm_Vertical" H 6550 5050 50  0001 C CNN
 F 3 "~" H 6550 5050 50  0001 C CNN
 	1    6550 5050
@@
 F 0 "J5" H 1168 4017 50  0000 C CNN
 F 1 "Conn_01x03" H 1168 3926 50  0000 C CNN
-F 2 "" H 1250 3700 50  0001 C CNN
+F 2 "Connector_JST:JST_XH_B03B-XH-A_1x03_P2.50mm_Vertical" H 1250 3700 50  0001 C CNN
 F 3 "~" H 1250 3700 50  0001 C CNN
 	1    1250 3700
@@
 F 0 "J7" H 9180 1392 50  0000 L CNN
 F 1 "Conn_01x02" H 9180 1301 50  0000 L CNN
-F 2 "" H 9100 1400 50  0001 C CNN
+F 2 "Connector_JST:JST_XH_B02B-XH-A_1x02_P2.50mm_Vertical" H 9100 1400 50  0001 C CNN
 F 3 "~" H 9100 1400 50  0001 C CNN
 	1    9100 1400

Commit message: Finish footprints.
Parts:
- C1, C2, C4, C5, C9: footprint (none) -> Capacitor_THT:C_Rect_L7.2mm_W5.5mm_P5.00mm_FKS2_FKP2_MKS2_MKP2
- C3: footprint (none) -> Capacitor_THT:C_Rect_L7.0mm_W2.0mm_P5.00mm
- C6, C7, C8: footprint (none) -> Capacitor_THT:C_Radial_D12.5mm_H25.0mm_P5.00mm
Changed lines of the file:
@@
 F 0 "C8" H 8018 2696 50  0000 L CNN
 F 1 "1m" H 8018 2605 50  0000 L CNN
-F 2 "" H 7938 2500 50  0001 C CNN
+F 2 "Capacitor_THT:C_Radial_D12.5mm_H25.0mm_P5.00mm" H 7938 2500 50  0001 C CNN
 F 3 "~" H 7900 2650 50  0001 C CNN
 	1    7900 2650
@@
 F 0 "C7" H 7668 2696 50  0000 L CNN
 F 1 "1m" H 7668 2605 50  0000 L CNN
-F 2 "" H 7588 2500 50  0001 C CNN
+F 2 "Capacitor_THT:C_Radial_D12.5mm_H25.0mm_P5.00mm" H 7588 2500 50  0001 C CNN
 F 3 "~" H 7550 2650 50  0001 C CNN
 	1    7550 2650
@@
 F 0 "C5" H 6718 2696 50  0000 L CNN
 F 1 "1u" H 6718 2605 50  0000 L CNN
-F 2 "" H 6638 2500 50  0001 C CNN
+F 2 "Capacitor_THT:C_Rect_L7.2mm_W5.5mm_P5.00mm_FKS2_FKP2_MKS2_MKP2" H 6638 2500 50  0001 C CNN
 F 3 "~" H 6600 2650 50  0001 C CNN
 	1    6600 2650
@@
 F 0 "C6" H 7268 2696 50  0000 L CNN
 F 1 "1m" H 7268 2605 50  0000 L CNN
-F 2 "" H 7188 2500 50  0001 C CNN
+F 2 "Capacitor_THT:C_Radial_D12.5mm_H25.0mm_P5.00mm" H 7188 2500 50  0001 C CNN
 F 3 "~" H 7150 2650 50  0001 C CNN
 	1    7150 2650
@@
 F 0 "C4" H 4665 3946 50  0000 L CNN
 F 1 "1u" H 4665 3855 50  0000 L CNN
-F 2 "" H 4588 3750 50  0001 C CNN
+F 2 "Capacitor_THT:C_Rect_L7.2mm_W5.5mm_P5.00mm_FKS2_FKP2_MKS2_MKP2" H 4588 3750 50  0001 C CNN
 F 3 "~" H 4550 3900 50  0001 C CNN
 	1    4550 3900
@@
 F 0 "C3" H 4315 3946 50  0000 L CNN
 F 1 "1n" H 4315 3855 50  0000 L CNN
-F 2 "" H 4238 3750 50  0001 C CNN
+F 2 "Capacitor_THT:C_Rect_L7.0mm_W2.0mm_P5.00mm" H 4238 3750 50  0001 C CNN
 F 3 "~" H 4200 3900 50  0001 C CNN
 	1    4200 3900
@@
 F 0 "C1" H 3065 1596 50  0000 L CNN
 F 1 "470n" H 3065 1505 50  0000 L CNN
-F 2 "" H 2988 1400 50  0001 C CNN
+F 2 "Capacitor_THT:C_Rect_L7.2mm_W5.5mm_P5.00mm_FKS2_FKP2_MKS2_MKP2" H 2988 1400 50  0001 C CNN
 F 3 "~" H 2950 1550 50  0001 C CNN
 	1    2950 1550
@@
 F 0 "C2" H 4215 1596 50  0000 L CNN
 F 1 "100n" H 4215 1505 50  0000 L CNN
-F 2 "" H 4138 1400 50  0001 C CNN
+F 2 "Capacitor_THT:C_Rect_L7.2mm_W5.5mm_P5.00mm_FKS2_FKP2_MKS2_MKP2" H 4138 1400 50  0001 C CNN
 F 3 "~" H 4100 1550 50  0001 C CNN
 	1    4100 1550
@@
 F 0 "C9" H 4765 4996 50  0000 L CNN
 F 1 "1u" H 4765 4905 50  0000 L CNN
-F 2 "" H 4688 4800 50  0001 C CNN
+F 2 "Capacitor_THT:C_Rect_L7.2mm_W5.5mm_P5.00mm_FKS2_FKP2_MKS2_MKP2" H 4688 4800 50  0001 C CNN
 F 3 "~" H 4650 4950 50  0001 C CNN
 	1    4650 4950
